File: regSMD/reg.kicad_pcb (KiCad board)
At the start: 2 copper layers, 100 x 81 mm, 280 parts, among them Q101 2N3904, Q102 2N3904, Q103 2N3904, Q104 2N3904, Q201 2N3904, Q202 2N3904, Q203 2N3904, Q204 2N3904, Q205 2N3904, Q206 2N3904, Q207 2N3904, Q208 2N3904, Q209 2N3904, Q210 2N3904, Q211 2N3904, Q212 2N3904, Q301 2N3904, Q302 2N3904, Q303 2N3904, Q304 2N3904, Q305 2N3904, Q306 2N3904, Q307 2N3904, Q308 2N3904, Q309 2N3904, Q310 2N3904, Q311 2N3904, Q312 2N3904, Q401 2N3904, Q402 2N3904, Q403 2N3904, Q404 2N3904, Q405 2N3904, Q406 2N3904, Q407 2N3904, Q408 2N3904, Q409 2N3904, Q410 2N3904, Q411 2N3904, Q412 2N3904, Q501 2N3904, Q502 2N3904, Q503 2N3904, Q504 2N3904, Q505 2N3904, Q506 2N3904, Q507 2N3904, Q508 2N3904, Q509 2N3904, Q510 2N3904, Q511 2N3904, Q512 2N3904, Q601 2N3904, Q602 2N3904, Q603 2N3904, Q604 2N3904, Q605 2N3904, Q606 2N3904, Q607 2N3904, Q608 2N3904, Q609 2N3904, Q610 2N3904, Q611 2N3904, Q612 2N3904, Q701 2N3904, Q702 2N3904, Q703 2N3904, Q704 2N3904, Q705 2N3904, Q706 2N3904, Q707 2N3904, Q708 2N3904, Q709 2N3904, Q710 2N3904, Q711 2N3904, Q712 2N3904, Q801 2N3904, Q802 2N3904, Q803 2N3904, Q804 2N3904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

Commit message: fixed 8bit reg v3 pcb
Routing:
- net GND: track 1058.7 -> 681.3 mm, vias 79 -> 44
- net +5V: track 525.0 -> 385.0 mm
- net Net-(Q503-B): track 130.7 -> 43.7 mm, vias 9 -> 3
- net Net-(Q903-B): track 130.7 -> 43.7 mm, vias 9 -> 3
- net Net-(Q603-B): track 130.7 -> 43.7 mm, vias 9 -> 3
- net Net-(Q303-B): track 130.7 -> 43.7 mm, vias 9 -> 3
- net Net-(Q803-B): track 130.7 -> 43.7 mm, vias 9 -> 3
- net Net-(Q403-B): track 130.7 -> 44.1 mm, vias 9 -> 3
- net Net-(Q703-B): track 130.7 -> 45.0 mm, vias 9 -> 3
- net Net-(Q401-B): track 121.9 -> 40.6 mm
- net Net-(Q801-B): track 121.9 -> 40.6 mm
- net Net-(Q501-B): track 121.9 -> 40.6 mm
- net Net-(Q301-B): track 121.9 -> 40.6 mm
- net Net-(Q901-B): track 121.9 -> 40.6 mm
- net Net-(Q701-B): track 121.9 -> 40.6 mm
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