File: pcb/regv4/dflipfop.kicad_sch (KiCad schematic)
At the start: 49 parts, among them Q201 MMBT3904, Q202 MMBT3904, Q203 MMBT3904, Q204 MMBT3904, Q207 MMBT3904, Q208 MMBT3904, Q209 MMBT3904, Q210 MMBT3904, Q211 MMBT3904, Q212 MMBT3904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

Commit message: regv4 rst
Parts:
- added Q1, Q17, Q2: MMBT3904, Package_TO_SOT_SMD:SOT-23, symbol Transistor_BJT:MMBT3904
- added R1, R2, R33: 10000, Resistor_SMD:R_0805_2012Metric, symbol Device:R
- added R17, R25: 4700, Resistor_SMD:R_0805_2012Metric, symbol Device:R
Connections:
- net +5V: now also R17.1, R25.1; no longer Q217.3 (C), Q218.3 (C), R210.1, R224.1, R226.2
- net GND: now also Q1.2 (E), Q17.2 (E), Q2.2 (E)
- net at Q209.3 (C), Q210.3 (C), R214.2: now also R2.1; no longer R201.1
- new net: Q2.1 (B), R2.2
- new net: Q1.3 (C), Q2.3 (C), R17.2, R33.1
- new net: Q217.3 (C), Q218.3 (C), R210.1, R224.1, R226.2
- new net: Q17.1 (B), R33.2
- new net: Q17.3 (C), R201.1, R25.2
- new net: Q1.1 (B), R1.2
- new net RST: R1.1
