File: pcb/regv4/regv4.kicad_pcb (KiCad board)
At the start: 2 copper layers, 406 parts, among them J101 DATA_IN, J102 DATA_OUT, J103 WR_EN, J104 CLK, J105 +5V, J106 GND, Q101 MMBT3904, Q102 MMBT3904, Q103 MMBT3904, Q201 MMBT3904, Q202 MMBT3904, Q203 MMBT3904, Q204 MMBT3904, Q207 MMBT3904, Q208 MMBT3904, Q209 MMBT3904, Q210 MMBT3904, Q211 MMBT3904, Q212 MMBT3904, Q213 MMBT3904, Q214 MMBT3904, Q215 MMBT3904, Q216 MMBT3904, Q217 MMBT3904, Q218 MMBT3904, Q219 MMBT3904, Q220 MMBT3904, Q221 MMBT3904, Q301 MMBT3904, Q302 MMBT3904, Q303 MMBT3904, Q304 MMBT3904, Q305 MMBT3904, Q306 MMBT3904, Q307 MMBT3904, Q308 MMBT3904, Q309 MMBT3904, Q310 MMBT3904, Q311 MMBT3904, Q312 MMBT3904, Q313 MMBT3904, Q314 MMBT3904, Q315 MMBT3904, Q316 MMBT3904, Q317 MMBT3904, Q318 MMBT3904, Q319 MMBT3904, Q401 MMBT3904, Q402 MMBT3904, Q403 MMBT3904, Q404 MMBT3904, Q405 MMBT3904, Q406 MMBT3904, Q407 MMBT3904, Q408 MMBT3904, Q409 MMBT3904, Q410 MMBT3904, Q411 MMBT3904, Q412 MMBT3904, Q413 MMBT3904, Q414 MMBT3904, Q415 MMBT3904, Q416 MMBT3904, Q417 MMBT3904, Q418 MMBT3904, Q419 MMBT3904, Q501 MMBT3904, Q502 MMBT3904, Q503 MMBT3904, Q504 MMBT3904, Q505 MMBT3904, Q506 MMBT3904, Q507 MMBT3904, Q508 MMBT3904, Q509 MMBT3904, Q510 MMBT3904, Q511 MMBT3904, Q512 MMBT3904, Q513 MMBT3904, Q514 MMBT3904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

Commit message: regv4 rst
Parts:
- added J1: RST, Connector_PinHeader_2.54mm:PinHeader_1x01_P2.54mm_Vertical, F.Cu at (63.5, 168.4)
- added Q1: MMBT3904, Package_TO_SOT_SMD:SOT-23, F.Cu at (147.6, 128.1)
- added Q10: MMBT3904, Package_TO_SOT_SMD:SOT-23, F.Cu at (147.6, 46.4)
- added Q11: MMBT3904, Package_TO_SOT_SMD:SOT-23, F.Cu at (32.4, 25.9)
- added Q12: MMBT3904, Package_TO_SOT_SMD:SOT-23, F.Cu at (32.4, 30.4)
- added Q13: MMBT3904, Package_TO_SOT_SMD:SOT-23, F.Cu at (103.9, 70.7)
- added Q14: MMBT3904, Package_TO_SOT_SMD:SOT-23, F.Cu at (103.9, 75.1)
- added Q15: MMBT3904, Package_TO_SOT_SMD:SOT-23, F.Cu at (103.9, 99.3)
- added Q16: MMBT3904, Package_TO_SOT_SMD:SOT-23, F.Cu at (103.9, 103.8)
- added Q17: MMBT3904, Package_TO_SOT_SMD:SOT-23, F.Cu at (147.6, 136.9)
- added Q18: MMBT3904, Package_TO_SOT_SMD:SOT-23, F.Cu at (103.9, 136.9)
- added Q19: MMBT3904, Package_TO_SOT_SMD:SOT-23, F.Cu at (147.6, 108.2)
- added Q2: MMBT3904, Package_TO_SOT_SMD:SOT-23, F.Cu at (147.6, 132.5)
- added Q20: MMBT3904, Package_TO_SOT_SMD:SOT-23, F.Cu at (147.6, 79.5)
- added Q21: MMBT3904, Package_TO_SOT_SMD:SOT-23, F.Cu at (147.6, 50.9)
- added Q22: MMBT3904, Package_TO_SOT_SMD:SOT-23, F.Cu at (32.4, 34.8)
- added Q23: MMBT3904, Package_TO_SOT_SMD:SOT-23, F.Cu at (103.9, 79.5)
- added Q24: MMBT3904, Package_TO_SOT_SMD:SOT-23, F.Cu at (103.9, 108.2)
- added Q25: MMBT3904, Package_TO_SOT_SMD:SOT-23, F.Cu at (58.8, 168.3)
- added Q26: MMBT3904, Package_TO_SOT_SMD:SOT-23, F.Cu at (58.8, 172.8)
- added Q3: MMBT3904, Package_TO_SOT_SMD:SOT-23, F.Cu at (103.9, 128.1)
- added Q4: MMBT3904, Package_TO_SOT_SMD:SOT-23, F.Cu at (103.9, 132.5)
- added Q5: MMBT3904, Package_TO_SOT_SMD:SOT-23, F.Cu at (147.6, 99.3)
- added Q6: MMBT3904, Package_TO_SOT_SMD:SOT-23, F.Cu at (147.6, 103.8)
- added Q7: MMBT3904, Package_TO_SOT_SMD:SOT-23, F.Cu at (147.6, 70.7)
- added Q8: MMBT3904, Package_TO_SOT_SMD:SOT-23, F.Cu at (147.6, 75.1)
- added Q9: MMBT3904, Package_TO_SOT_SMD:SOT-23, F.Cu at (147.6, 42.0)
- added R1: 10000, Resistor_SMD:R_0805_2012Metric, F.Cu at (166.9, 127.3)
- added R10: 10000, Resistor_SMD:R_0805_2012Metric, F.Cu at (166.9, 44.1)
- added R11: 10000, Resistor_SMD:R_0805_2012Metric, F.Cu at (51.8, 25.1)
- added R12: 10000, Resistor_SMD:R_0805_2012Metric, F.Cu at (51.8, 28.1)
- added R13: 10000, Resistor_SMD:R_0805_2012Metric, F.Cu at (123.3, 69.9)
- added R14: 10000, Resistor_SMD:R_0805_2012Metric, F.Cu at (123.3, 72.8)
- added R15: 10000, Resistor_SMD:R_0805_2012Metric, F.Cu at (123.3, 98.6)
- added R16: 10000, Resistor_SMD:R_0805_2012Metric, F.Cu at (123.3, 101.5)
- added R17: 4700, Resistor_SMD:R_0805_2012Metric, F.Cu at (166.9, 133.2)
- added R18: 4700, Resistor_SMD:R_0805_2012Metric, F.Cu at (123.3, 133.2)
- added R19: 4700, Resistor_SMD:R_0805_2012Metric, F.Cu at (166.9, 104.5)
- added R2: 10000, Resistor_SMD:R_0805_2012Metric, F.Cu at (166.9, 130.2)
- added R20: 4700, Resistor_SMD:R_0805_2012Metric, F.Cu at (166.9, 75.8)
- added R21: 4700, Resistor_SMD:R_0805_2012Metric, F.Cu at (166.9, 47.1)
- added R22: 4700, Resistor_SMD:R_0805_2012Metric, F.Cu at (53.0, 62.0)
- added R23: 4700, Resistor_SMD:R_0805_2012Metric, F.Cu at (123.3, 75.8)
- added R24: 4700, Resistor_SMD:R_0805_2012Metric, F.Cu at (123.3, 104.5)
- added R25: 4700, Resistor_SMD:R_0805_2012Metric, F.Cu at (166.9, 136.2)
- added R26: 4700, Resistor_SMD:R_0805_2012Metric, F.Cu at (123.3, 136.2)
- added R27: 4700, Resistor_SMD:R_0805_2012Metric, F.Cu at (166.9, 107.5)
- added R28: 4700, Resistor_SMD:R_0805_2012Metric, F.Cu at (166.9, 78.8)
- added R29: 4700, Resistor_SMD:R_0805_2012Metric, F.Cu at (166.9, 50.0)
- added R3: 10000, Resistor_SMD:R_0805_2012Metric, F.Cu at (123.3, 127.3)
- added R30: 4700, Resistor_SMD:R_0805_2012Metric, F.Cu at (53.0, 59.0)
- added R31: 4700, Resistor_SMD:R_0805_2012Metric, F.Cu at (123.3, 78.8)
- added R32: 4700, Resistor_SMD:R_0805_2012Metric, F.Cu at (123.3, 107.5)
- added R33: 10000, Resistor_SMD:R_0805_2012Metric, F.Cu at (166.9, 139.1)
- added R34: 10000, Resistor_SMD:R_0805_2012Metric, F.Cu at (123.3, 139.1)
- added R35: 10000, Resistor_SMD:R_0805_2012Metric, F.Cu at (166.9, 110.4)
- added R36: 10000, Resistor_SMD:R_0805_2012Metric, F.Cu at (166.9, 81.7)
- added R37: 10000, Resistor_SMD:R_0805_2012Metric, F.Cu at (166.9, 53.0)
- added R38: 10000, Resistor_SMD:R_0805_2012Metric, F.Cu at (51.8, 37.0)
- added R39: 10000, Resistor_SMD:R_0805_2012Metric, F.Cu at (123.3, 81.7)
- added R4: 10000, Resistor_SMD:R_0805_2012Metric, F.Cu at (123.3, 130.2)
- added R40: 10000, Resistor_SMD:R_0805_2012Metric, F.Cu at (123.3, 110.4)
- added R41: 4700, Resistor_SMD:R_0805_2012Metric, F.Cu at (49.3, 158.7)
- added R42: 10000, Resistor_SMD:R_0805_2012Metric, F.Cu at (49.3, 161.7)
- added R43: 4700, Resistor_SMD:R_0805_2012Metric, F.Cu at (49.3, 164.6)
- added R44: 10000, Resistor_SMD:R_0805_2012Metric, F.Cu at (53.7, 158.7)
- added R5: 10000, Resistor_SMD:R_0805_2012Metric, F.Cu at (166.9, 98.6)
- added R6: 10000, Resistor_SMD:R_0805_2012Metric, F.Cu at (166.9, 101.5)
- added R7: 10000, Resistor_SMD:R_0805_2012Metric, F.Cu at (166.9, 69.9)
- added R8: 10000, Resistor_SMD:R_0805_2012Metric, F.Cu at (166.9, 72.8)
- added R9: 10000, Resistor_SMD:R_0805_2012Metric, F.Cu at (166.9, 41.2)
- moved R624 105.9 mm to (184.6, 41.2)
- moved R617 104.5 mm to (180.2, 41.2)
- moved R618 104.5 mm to (180.2, 44.1)
- moved Q101 103.6 mm to (58.8, 177.2)
- moved Q102 103.6 mm to (58.8, 181.7)
- moved Q103 103.6 mm to (58.8, 186.1)
- moved R610 103.2 mm to (175.8, 41.2)
- moved R611 103.2 mm to (175.8, 44.1)
- moved R612 103.2 mm to (175.8, 47.1)
- moved Q610 102.6 mm to (157.4, 42.0)
- moved R603 102.0 mm to (171.4, 41.2)
- moved R606 102.0 mm to (171.4, 50.0)
- moved R604 102.0 mm to (171.4, 44.1)
- moved R605 102.0 mm to (171.4, 47.1)
- moved Q604 99.6 mm to (152.5, 42.0)
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Connections:
- Q217 pad 3: +5V -> Net-(Q217-C)
- Q218 pad 3: +5V -> Net-(Q217-C)
- Q317 pad 3: +5V -> Net-(Q317-C)
- Q319 pad 3: +5V -> Net-(Q317-C)
- Q417 pad 3: +5V -> Net-(Q417-C)
- Q419 pad 3: +5V -> Net-(Q417-C)
- Q517 pad 3: +5V -> Net-(Q517-C)
- Q519 pad 3: +5V -> Net-(Q517-C)
- Q617 pad 3: +5V -> Net-(Q617-C)
- Q619 pad 3: +5V -> Net-(Q617-C)
- Q717 pad 3: +5V -> Net-(Q717-C)
- Q719 pad 3: +5V -> Net-(Q717-C)
- Q817 pad 3: +5V -> Net-(Q817-C)
- Q819 pad 3: +5V -> Net-(Q817-C)
- Q917 pad 3: +5V -> Net-(Q917-C)
- Q919 pad 3: +5V -> Net-(Q917-C)
- R201 pad 1: Net-(Q209-C) -> Net-(Q17-C)
- R210 pad 1: +5V -> Net-(Q217-C)
- R224 pad 1: +5V -> Net-(Q217-C)
- R226 pad 2: +5V -> Net-(Q217-C)
- R312 pad 1: +5V -> Net-(Q317-C)
- R319 pad 1: Net-(Q301-C) -> Net-(Q18-C)
- R324 pad 1: +5V -> Net-(Q317-C)
- R328 pad 2: +5V -> Net-(Q317-C)
- R412 pad 1: +5V -> Net-(Q417-C)
- R419 pad 1: Net-(Q401-C) -> Net-(Q19-C)
- R424 pad 1: +5V -> Net-(Q417-C)
- R428 pad 2: +5V -> Net-(Q417-C)
- R512 pad 1: +5V -> Net-(Q517-C)
- R519 pad 1: Net-(Q501-C) -> Net-(Q20-C)
- R524 pad 1: +5V -> Net-(Q517-C)
- R528 pad 2: +5V -> Net-(Q517-C)
- R612 pad 1: +5V -> Net-(Q617-C)
- R619 pad 1: Net-(Q601-C) -> Net-(Q21-C)
- R624 pad 1: +5V -> Net-(Q617-C)
- R628 pad 2: +5V -> Net-(Q617-C)
- R712 pad 1: +5V -> Net-(Q717-C)
- R719 pad 1: Net-(Q701-C) -> Net-(Q22-C)
- R724 pad 1: +5V -> Net-(Q717-C)
- R728 pad 2: +5V -> Net-(Q717-C)
- R812 pad 1: +5V -> Net-(Q817-C)
- R819 pad 1: Net-(Q801-C) -> Net-(Q23-C)
- R824 pad 1: +5V -> Net-(Q817-C)
- R828 pad 2: +5V -> Net-(Q817-C)
- R912 pad 1: +5V -> Net-(Q917-C)
- R919 pad 1: Net-(Q901-C) -> Net-(Q24-C)
- R924 pad 1: +5V -> Net-(Q917-C)
- R928 pad 2: +5V -> Net-(Q917-C)
Routing:
- net +5V: track 0.00 -> 35.5 mm

Commit message: small work on regv4 (so lazy)
Parts:
- removed Q10, Q11, Q12, Q13, Q14, Q15, Q16, Q21, Q22, Q23, Q24, Q601, Q602, Q603, Q604, Q605, Q606, Q607, Q608, Q609, Q610, Q611, Q612, Q613, Q614, Q615, Q616, Q617, Q618, Q619, Q701, Q702, Q703, Q704, Q705, Q706, Q707, Q708, Q709, Q710, Q711, Q712, Q713, Q714, Q715, Q716, Q717, Q718, Q719, Q801, Q802, Q803, Q804, Q805, Q806, Q807, Q808, Q809, Q810, Q811, Q812, Q813, Q814, Q815, Q816, Q817, Q818, Q819, Q9, Q901, Q902, Q903, Q904, Q905, Q906, Q907, Q908, Q909, Q910, Q911, Q912, Q913, Q914, Q915, Q916, Q917, Q918, Q919: MMBT3904, Package_TO_SOT_SMD:SOT-23
- removed R10, R11, R12, R13, R14, R15, R16, R37, R38, R39, R40, R601, R602, R603, R605, R609, R610, R611, R612, R614, R617, R618, R619, R620, R623, R624, R625, R626, R629, R630, R701, R702, R703, R705, R709, R710, R711, R712, R714, R717, R718, R719, R720, R723, R724, R725, R726, R729, R730, R801, R802, R803, R805, R809, R810, R811, R812, R814, R817, R818, R819, R820, R823, R824, R825, R826, R829, R830, R9, R901, R902, R903, R905, R909, R910, R911, R912, R914, R917, R918, R919, R920, R923, R924, R925, R926, R929, R930: 10000, Resistor_SMD:R_0805_2012Metric
- removed R21, R22, R23, R24, R29, R30, R31, R32, R604, R606, R607, R608, R613, R615, R616, R621, R622, R627, R628, R704, R706, R707, R708, R713, R715, R716, R721, R722, R727, R728, R804, R806, R807, R808, R813, R815, R816, R821, R822, R827, R828, R904, R906, R907, R908, R913, R915, R916, R921, R922, R927, R928: 4700, Resistor_SMD:R_0805_2012Metric
- J101: value DATA_IN -> Conn_01x04_Pin; footprint Connector_PinHeader_2.54mm:PinHeader_1x08_P2.54mm_Vertical -> Connector_PinHeader_2.54mm:PinHeader_1x04_P2.54mm_Vertical
- J102: value DATA_OUT -> Conn_01x04_Pin; footprint Connector_PinHeader_2.54mm:PinHeader_1x08_P2.54mm_Vertical -> Connector_PinHeader_2.54mm:PinHeader_1x04_P2.54mm_Vertical
- moved Q512 132.5 mm to (34.5, 29.8)
- moved Q513 132.5 mm to (34.5, 34.3)
- moved Q514 132.5 mm to (34.5, 38.7)
- moved Q515 132.5 mm to (34.5, 43.2)
- moved Q516 132.5 mm to (39.5, 20.9)
- moved Q517 132.5 mm to (39.5, 25.4)
- moved Q518 132.5 mm to (39.5, 29.8)
- moved Q519 132.5 mm to (39.5, 34.3)
- moved R36 132.5 mm to (44.1, 32.0)
- moved R501 132.5 mm to (44.1, 34.9)
- moved R502 132.5 mm to (44.1, 37.9)
- moved R510 132.5 mm to (52.9, 20.2)
- moved R511 132.5 mm to (52.9, 23.1)
- moved R512 132.5 mm to (52.9, 26.1)
- moved R514 132.5 mm to (52.9, 32.0)
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Routing:
- net +5V: track 35.5 -> 0.00 mm
Other:
- board outline added: 100 x 100 mm
- copper layers 2 -> 4
