File: pcb/regv4/regv4.kicad_sch (KiCad schematic)
At the start: 14 parts, among them J101 DATA_IN, J102 DATA_OUT, J103 WR_EN, J104 CLK, J105 +5V, J106 GND, Q101 MMBT3904, Q102 MMBT3904, Q103 MMBT3904

Commit message: regv4 rst
Parts:
- added J1: RST, Connector_PinHeader_2.54mm:PinHeader_1x01_P2.54mm_Vertical, symbol Connector:Conn_01x01_Pin
- added Q25, Q26: MMBT3904, Package_TO_SOT_SMD:SOT-23, symbol Transistor_BJT:MMBT3904
- added R41, R43: 4700, Resistor_SMD:R_0805_2012Metric, symbol Device:R
- added R42, R44: 10000, Resistor_SMD:R_0805_2012Metric, symbol Device:R
Connections:
- net +5V: now also R41.1, R43.1
- net GND: now also Q25.2 (E), Q26.2 (E)
- new net: Q25.3 (C), R41.2, R44.1
- new net: Q26.1 (B), R44.2
- new net: Q25.1 (B), R42.2
- new net: J1.1 (Pin_1), R42.1
- new net RST: Q26.3 (C), R43.2

Commit message: small work on regv4 (so lazy)
Parts:
- removed J101: DATA_IN, Connector_PinHeader_2.54mm:PinHeader_1x08_P2.54mm_Vertical, symbol Connector:Conn_01x08_Pin
- removed J102: DATA_OUT, Connector_PinHeader_2.54mm:PinHeader_1x08_P2.54mm_Vertical, symbol Connector:Conn_01x08_Pin
- added J101, J102: Conn_01x04_Pin, Connector_PinHeader_2.54mm:PinHeader_1x04_P2.54mm_Vertical, symbol Connector:Conn_01x04_Pin
Connections:
- net DFlipFlop/Data: now also J101.1 (Pin_1)
- net DFlipFlop/Q: now also J102.1 (Pin_1)
- net DFlipFlop1/Data: now also J101.2 (Pin_2)
- net DFlipFlop1/Q: now also J102.2 (Pin_2)
- net DFlipFlop2/Data: now also J101.3 (Pin_3)
- net DFlipFlop2/Q: now also J102.3 (Pin_3)
- net DFlipFlop3/Data: now also J101.4 (Pin_4)
- net DFlipFlop3/Q: now also J102.4 (Pin_4)
Other:
- removed sheet DFlipFlop4
- removed sheet DFlipFlop5
- removed sheet DFlipFlop6
- removed sheet DFlipFlop7
